File: coffeepowersupply.sch (KiCad schematic (older format))
At the start: 37 parts, among them J1 Conn_01x03_Male, J2 Conn_01x02_Male, J3 Conn_01x02_Male, J4 Conn_01x02_Male, Q1 BT139-600, Q2 BT139-600, U1 MOC3021, U2 PC817, U3 PC817, U4 MOC3021

Commit message: Add files via upload
Parts:
- added C?: 10n, symbol Device:C
- added C?: 200u, symbol Device:C
- added U?: STM32F030C8Tx, Package_QFP:LQFP-48_7x7mm_P0.5mm, symbol MCU_ST_STM32F0:STM32F030C8Tx
Connections:
- net +V: now also C?.1, C?.1, U?.1 (VDD), U?.11 (PA1), U?.24 (VDD), U?.48 (VDD), U?.9 (VDDA)
- net BoilerMCU: now also U?.12 (PA2)
- net NTC: now also U?.10 (PA0)
- net Pump_MCU: now also U?.13 (PA3)
- net MCU renamed Null_MCU
- net Null_MCU: now also U?.14 (PA4)
- new net SWCLK: U?.37 (PA14)
- new net SWDIO: U?.34 (PA13)
- new net VSS: C?.2, U?.23 (VSS), U?.47 (VSS)
- new net VSSA: C?.2, U?.8 (VSSA)
Other:
- note added: "PS Filter\nAs Close as \npossible to MCU\n"
Changed lines of the file:
@@
 	6250 6600 6550 6600
 Text Label 6550 6600 0    50   ~ 0
-MCU
+Null_MCU
 $Comp
 L Device:R R7
@@
 Wire Notes Line
 	8700 4800 3750 4800
+$Comp
+L MCU_ST_STM32F0:STM32F030C8Tx U?
+U 1 1 60188C82
+P 1350 4300
+F 0 "U?" H 1350 2611 50  0000 C CNN
+F 1 "STM32F030C8Tx" H 1350 2520 50  0000 C CNN
+F 2 "Package_QFP:LQFP-48_7x7mm_P0.5mm" H 850 2800 50  0001 R CNN
+F 3 "http://www.st.com/st-web-ui/static/active/en/resource/technical/document/datasheet/DM00088500.pdf" H 1350 4300 50  0001 C CNN
+	1    1350 4300
+	1    0    0    -1
+$EndComp
+Wire Wire Line
+	1950 5500 2500 5500
+Wire Wire Line
+	1950 5600 2500 5600
+Text Label 2500 5500 0    50   ~ 0
+SWDIO
+Text Label 2500 5600 0    50   ~ 0
+SWCLK
+$Comp
+L Device:C C?
+U 1 1 601959AB
+P 850 6800
+F 0 "C?" H 965 6846 50  0000 L CNN
+F 1 "10n" H 965 6755 50  0000 L CNN
+F 2 "" H 888 6650 50  0001 C CNN
+F 3 "~" H 850 6800 50  0001 C CNN
+	1    850  6800
+	1    0    0    -1
+$EndComp
+$Comp
+L Device:C C?
+U 1 1 601A92CE
+P 850 7450
+F 0 "C?" H 965 7496 50  0000 L CNN
+F 1 "200u" H 965 7405 50  0000 L CNN
+F 2 "" H 888 7300 50  0001 C CNN
+F 3 "~" H 850 7450 50  0001 C CNN
+	1    850  7450
+	1    0    0    -1
+$EndComp
+Wire Wire Line
+	1550 2700 1550 2550
+Text Label 1550 2550 0    50   ~ 0
+VDDA
+Wire Wire Line
+	1450 5900 1450 6300
+Text Label 1450 6300 0    50   ~ 0
+VSSA
+Text Label 600  6550 0    50   ~ 0
++V
+Text Label 1050 6550 0    50   ~ 0
+VDDA
+Wire Wire Line
+	600  6550 850  6550
+Wire Wire Line
+	850  6550 850  6650
+Wire Wire Line
+	850  6550 1050 6550
+Connection ~ 850  6550
+Wire Wire Line
+	850  6950 850  7050
+Text Label 850  7050 0    50   ~ 0
+VSSA
+Wire Wire Line
+	850  7300 850  7250
+Wire Wire Line
+	850  7250 1150 7250
+Wire Wire Line
+	850  7250 650  7250
+Connection ~ 850  7250
+Text Label 650  7250 0    50   ~ 0
++V
+Text Label 1150 7250 0    50   ~ 0
+VDD
+Wire Wire Line
+	1250 2700 1250 2550
+Text Label 1250 2550 0    50   ~ 0
+VDD
+Wire Wire Line
+	850  7600 850  7750
+Wire Wire Line
+	850  7750 1050 7750
+Wire Wire Line
+	1250 5900 1250 6000
+Wire Wire Line
+	1250 6000 1350 6000
+Wire Wire Line
+	1350 6000 1350 5900
+Text Label 1250 6000 0    50   ~ 0
+VSS
+Text Label 1050 7750 0    50   ~ 0
+VSS
+Wire Wire Line
+	1450 2700 1450 2600
+Wire Wire Line
+	1450 2600 1350 2600
+Wire Wire Line
+	1350 2600 1350 2700
+Wire Wire Line
+	1250 2550 1350 2550
+Wire Wire Line
+	1350 2550 1350 2600
+Connection ~ 1350 2600
+Wire Notes Line
+	550  6450 550  7800
+Wire Notes Line
+	1850 7800 1850 6450
+Wire Notes Line
+	550  6450 1850 6450
+Wire Notes Line
+	550  7800 1850 7800
+Text Notes 1200 6900 0    50   ~ 0
+PS Filter\nAs Close as \npossible to MCU\n
+Wire Wire Line
+	1950 4200 2300 4200
+Text Label 2300 4200 0    50   ~ 0
+NTC
+Wire Wire Line
+	1950 4400 2300 4400
+Wire Wire Line
+	1950 4500 2300 4500
+Text Label 2300 4400 0    50   ~ 0
+BoilerMCU
+Text Label 2300 4500 0    50   ~ 0
+Pump_MCU
+Wire Wire Line
+	1950 4600 2300 4600
+Text Label 2300 4600 0    50   ~ 0
+Null_MCU
+Text Label 7900 5450 0    50   ~ 0
+FlowmeterMCU
+Wire Wire Line
+	1950 4300 2300 4300
+Text Label 2300 4300 0    50   ~ 0
+FlowmeterMCU
 $EndSCHEMATC

Commit message: Add files via upload
Parts:
- added C? (x2): 0.1u, symbol Device:C
- added C?: 220u, symbol Device:CP
- added C? (x2): 100n, symbol Device:C
- added J5: Conn_01x04_Male, symbol Connector:Conn_01x04_Male
- added R? (x2): 10k, symbol Device:R
- C9: renamed from C?; value 200u -> 100n
- gave numbers to parts that had none: 2
Connections:
- net VSS is gone; now on net GND: C9.2, U5.23 (VSS), U5.47 (VSS)
- net VSSA is gone; now on net GND: C8.2, U5.8 (VSSA)
- net GND: now also C?.1, C?.2, C?.2, C?.2, C?.2, J5.4 (Pin_4), R?.1
- net SWCLK: now also J5.3 (Pin_3)
- net SWDIO: now also J5.2 (Pin_2)
- net at U5.44 (BOOT0): now also R?.2
- net at U5.7 (NRST): now also C?.2, R?.2
- net FlowmeterMCU: now reaches D1.2 (A), D2.1 (K), J1.1 (Pin_1), R12.2, R15.2
- net FlowmeterMCU: now also U5.11 (PA1)
- net +V renamed +3V3
- net +3V3: now also C?.1, C?.1, C?.1, C?.1, J5.1 (Pin_1), R?.1; no longer U5.11 (PA1)
Other:
- note added: "MCU\n"
- note added: "PROG. Pins"
- moved on the sheet: C1, C2, C3, C4, C5, C6, C7, C8, C9, D1, D2, D3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
